File: boards/gardenprobe-c6/gardenprobe-c6.kicad_pcb (KiCad board)
At the start: 2 copper layers, 70 x 25 mm, 19 parts, among them J1 Conn_01x04, J2 SOIL_PROBE, Q1 AO3401A, U1 ESP32-C6-WROOM-1, U2 MCP1700-3302, U3 SHT31

Commit message: feat: add boards/gardenprobe-c6/gardenprobe-c6.kicad_pcb
Parts:
- R6: value (none) -> 4.7k
Changed lines of the file:
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@@
+          (thickness 0.15)
+        )
+      )
+    )
+    (property
+      "Value"
+      "4.7k"
+      (at 0 2 0)
+      (layer "F.Fab")
+      (effects
+        (font
+          (size 1 1)
           (thickness 0.15)
         )
