File: boards/relaymini-c3/relaymini-c3.kicad_pcb (KiCad board)
At the start: 2 copper layers, 60 x 40 mm, 39 parts, among them J1 Term_5.08_2P, J2 Term_5.08_2P, J3 Conn_01x04, K1 HF32F-G, Q1 S8050, U1 HLK-PM01, U2 AP2112K-3.3, U3 BL0942, U4 PC817, U5 PC817, U6 ESP32-C3-WROOM-02

Commit message: feat: add boards/relaymini-c3/relaymini-c3.kicad_pcb
Parts:
- R15: value (none) -> 10k
Changed lines of the file:
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@@
+          (size 1 1)
+          (thickness 0.15)
+        )
+      )
+    )
+    (property
+      "Value"
+      "10k"
+      (at 0 2 0)
+      (layer "F.Fab")
+      (effects
+        (font
           (size 1 1)
           (thickness 0.15)
